Commit message: Fixed_urdf

File: urdf/SCARA.urdf (robot description, URDF)
Before this commit: robot origins, 1 links, 0 joints
Links:
- added link link_1, mass 1; collision cylinder length=0.1 radius=0.5; visual cylinder length=0.2 radius=0.1
Joints:
- added joint joint1: type revolute, parent base_link, child link_1, origin xyz=0 0 0.1 rpy=0  0  0, axis 0  0  1, limit lower=-1.79769e+308 upper=1.79769e+308 effort=-1.0 velocity=-1.0

Commit message: Stuff

File: urdf/SCARA.urdf (robot description, URDF)
Before this commit: robot origins, 2 links, 1 joints
Links:
- added link link_2, mass 1; collision box size=1 1 1; visual box size=1 1 1
- added link link_3, mass 1; collision cylinder length=5 radius=0.5; visual cylinder length=5 radius=0.5
- link link_1: geometry collision cylinder length=4.9 radius=0.5; visual cylinder length=4.9 radius=0.5
Joints:
- removed joint joint1
- added joint joint_1: type revolute, parent base_link, child link_1, origin xyz=0 0 0.1 rpy=0  0  0, axis 0  0  1, limit lower=-1.79769e+308 upper=1.79769e+308 effort=-1.0 velocity=-1.0
- added joint joint_2: type fixed, parent link_1, child link_2, origin xyz=0 0 5.5 rpy=0    1.57  0, axis 0  0  0, limit lower=0 upper=0 effort=0 velocity=0
- added joint joint_3: type fixed, parent link_2, child link_3, origin xyz=2.99999  0       0 rpy=0    1.57  0, axis 0  0  0, limit lower=0 upper=0 effort=0 velocity=0

Commit message: fixed_flying links

File: urdf/SCARA.urdf (robot description, URDF)
Before this commit: robot origins, 4 links, 3 joints
Links:
- removed link link_3
- link base_link: mass 100 -> None; geometry collision box size=0 0 0; visual box size=0 0 0
- link link_1: geometry collision cylinder length=4.9 radius=0.5; visual cylinder length=5 radius=0.3
Joints:
- removed joint joint_3
- joint joint_1: origin xyz=0 0 0.1 rpy=0  0  0 -> xyz=0 0 1 rpy=0  0  0; type revolute -> fixed
- joint joint_2: type fixed -> revolute

Commit message: urdf ready

File: urdf/SCARA.urdf (robot description, URDF)
Before this commit: robot origins, 3 links, 2 joints
Links:
- added link link_3, mass 1; collision cylinder length=5 radius=0.3; visual cylinder length=5 radius=0.3
- added link link_4, mass 1; collision cylinder length=1 radius=0.5; visual cylinder length=1 radius=0.5
- added link link_5, mass 1; collision box size=1 1 1; visual box size=1 1 1
- added link link_6, mass 1; collision box size=1 1 0.2; visual box size=1 1 0.2
- link base_link: mass None -> 100
- link link_1: geometry collision cylinder length=5 radius=0.5; visual cylinder length=5 radius=0.3
Joints:
- added joint joint_3: type fixed, parent link_2, child link_3, origin xyz=3 0 0 rpy=0  1.57  0, axis 0  0  0, limit lower=0 upper=0 effort=0 velocity=0
- added joint joint_4: type fixed, parent link_3, child link_4, origin xyz=2.38000000e-03   0.00000000e+00   3.00000000e+00 rpy=0   -1.57  0, axis 0  0  0, limit lower=0 upper=0 effort=0 velocity=0
- added joint joint_5: type revolute, parent link_4, child link_5, origin xyz=1  0  0 rpy=0  0  0, axis 0  0  1, limit lower=-1.79769e+308 upper=1.79769e+308 effort=-1.0 velocity=-1.0
- added joint joint_6: type prismatic, parent link_5, child link_6, origin xyz=0       0      -0.6 rpy=0  0  0, axis 1  0  0, limit lower=-1.79769e+308 upper=1.79769e+308 effort=-1.0 velocity=-1.0
- joint joint_2: origin xyz=0 0 5.5 rpy=0    1.57  0 -> xyz=0 0 5.5 rpy=0  0  1

Commit message: Urdf is correct, just need to get joint_states to run correctly and we are almost all set

File: urdf/SCARA.urdf (robot description, URDF)
Before this commit: robot origins, 7 links, 6 joints
Links:
- removed link base_link
- added link world
- link link_6: geometry collision box size=0.5 0.5 4; visual box size=0.5 0.5 4
Joints:
- joint joint_1: limit lower=-1.79769e+308 upper=1.79769e+308 effort=-1.0 velocity=-1.0 -> (none); origin xyz=0 0 1 rpy=0  0  0 -> xyz=0 0 0 rpy=0  0  0; parent base_link -> world
- joint joint_2: axis 0  0  0 -> 0  0  1; limit lower=0 upper=0 effort=0 velocity=0 -> lower=-3.14 upper=3.14 effort=100 velocity=0
- joint joint_5: limit lower=-1.79769e+308 upper=1.79769e+308 effort=-1.0 velocity=-1.0 -> lower=-3.14 upper=3.14 effort=100 velocity=-1.0; origin xyz=1  0  0 rpy=0  0  0 -> xyz=0  0  0 rpy=0  0  0
- joint joint_6: axis 1  0  0 -> 0 0 -1; limit lower=-1.79769e+308 upper=1.79769e+308 effort=-1.0 velocity=-1.0 -> lower=-2 upper=2 effort=100 velocity=-1.0; origin xyz=0       0      -0.6 rpy=0  0  0 -> xyz=1       0      -0.6 rpy=0  0  0

Commit message: Supposed URDF changes? Might want to revert these but my computer is forcing me to push this to pull

File: urdf/SCARA.urdf (robot description, URDF)
Before this commit: robot origins, 3 links, 2 joints
Links:
- added link link_3, mass 1; collision cylinder length=5 radius=0.5; visual cylinder length=5 radius=0.5
Joints:
- added joint joint_3: type fixed, parent link_2, child link_3, origin xyz=0.5  0       5.5 rpy=0    1.57  0, axis 0  0  0, limit lower=0 upper=0 effort=0 velocity=0
