Commit message: PD controller almost done, just need to record the positions and send to MATLAB

File: urdf/SCARAFIXED.urdf (robot description, URDF)
Before this commit: robot origins, 7 links, 6 joints
Joints:
- joint joint_2: type revolute -> fixed

Commit message: fixed the wierd error

File: urdf/SCARAFIXED.urdf (robot description, URDF)
Before this commit: robot origins, 7 links, 6 joints
Joints:
- joint joint_5: type fixed -> revolute
- joint joint_6: type prismatic -> fixed

Commit message: velocity controller progress

File: urdf/SCARAFIXED.urdf (robot description, URDF)
Before this commit: robot origins, 7 links, 6 joints
Joints:
- joint joint_6: type fixed -> prismatic
