Commit message: changed 1s to 0s

File: urdf/SCARA2.urdf (robot description, URDF)
Before this commit: robot origins, 7 links, 6 joints
Joints:
- joint joint_2: limit lower=-3.14 upper=3.14 effort=1000000 velocity=1000000 -> lower=-31.4 upper=31.4 effort=1000000 velocity=1000000
- joint joint_5: limit lower=-3.14 upper=3.14 effort=1000000 velocity=1000000 -> lower=-31.4 upper=31.4 effort=1000000 velocity=1000000

Commit message: changes to urdf, fixed himje position and set lower joint limits

File: urdf/SCARA2.urdf (robot description, URDF)
Before this commit: robot origins, 7 links, 6 joints
Joints:
- joint joint_2: limit lower=-31.4 upper=31.4 effort=1000000 velocity=1000000 -> lower=-1 upper=1 effort=1000000 velocity=1000000; origin xyz=0 0 5.5 rpy=0  0  1 -> xyz=0 0 5.5 rpy=0  0  1.5708
- joint joint_5: limit lower=-31.4 upper=31.4 effort=1000000 velocity=1000000 -> lower=-1 upper=1 effort=1000000 velocity=1000000
